File: stepper_schematic/stepper.kicad_pcb (KiCad board)
At the start: 2 copper layers, 68 parts, among them IC1 ATMEGA8-P, IC2 SP485, IC3 LTV-814, IC4 LTV-814, IC5 LTV-814, IC6 LTV-814, IC7 LTV-814, IC8 LM2575, P1 CONN_6, P2 HN1X6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

Commit message: I forgot the changes and generate the pdf for documentation and schematics
Parts:
- IC8: value LM2575 -> LM2575_PENTAWATT_D2PAK
- JP1, JP2, JP3, JP4, JP5: value (none) -> JUMPER
- X1: value (none) -> QUARTZ
Connections:
- U1 pad 12: /RXD -> (no net)
- U1 pad 9: (no net) -> /RXD
Routing:
- net /RXD: track 35.8 -> 40.6 mm
Other:
- board text added: "DRV BIBA'S stepper motor V0.2"
- board text added: "STEPPER MOTOR V0.2"
- board text removed: "DRV BIBA'S stepper motor V0.1"
- board text removed: "STEPPER MOTOR V0.1"
